File: hw/GameBrian_v0.1/GameBrian_v0.1.kicad_sch (KiCad schematic)
At the start: 110 parts, among them J1 USB_C_Receptacle_USB2.0_16P, J2 GameBoy_GamePak_AGB-002, J3 Micro_SD_Card_Det_Hirose_DM3AT, J4 Debug, J5 Config, J6 GPIO, Q1 Q_NMOS_GSD, Q2 Q_NMOS_GSD, SW10 Program, SW8 Reset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

Commit message: Checkpoint (pre-final route)
Connections:
- net +3V3: no longer U1.N10 (CFG_0)
- net GND: now also U1.N10 (CFG_0)
- no-connect marks 4 -> 15
Other:
- moved on the sheet: C16, C17, C18, C19, C22, C23, C24, C25, U1C, U1D, U1F, U1G

Commit message: Checkpoint (DDR RAM?)
Other:
- moved on the sheet: C14, C15, U1B
Changed lines of the file:
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@@
 	)
 	(junction
-		(at 439.42 96.52)
+		(at 588.01 276.86)
 		(diameter 0)
 		(color 0 0 0 0)
@@
 	)
 	(junction
-		(at 443.23 91.44)
+		(at 591.82 271.78)
 		(diameter 0)
 		(color 0 0 0 0)
@@
 	)
 	(junction
-		(at 473.71 91.44)
+		(at 622.3 271.78)
 		(diameter 0)
 		(color 0 0 0 0)
@@
 	(wire
 		(pts
-			(xy 439.42 96.52) (xy 443.23 96.52)
+			(xy 588.01 276.86) (xy 591.82 276.86)
 		)
 		(stroke
@@
 	(wire
 		(pts
-			(xy 473.71 91.44) (xy 473.71 92.71)
+			(xy 622.3 271.78) (xy 622.3 273.05)
 		)
 		(stroke
@@
 	(wire
 		(pts
-			(xy 443.23 91.44) (xy 473.71 91.44)
+			(xy 591.82 271.78) (xy 622.3 271.78)
 		)
 		(stroke
@@
 	(wire
 		(pts
-			(xy 439.42 91.44) (xy 443.23 91.44)
+			(xy 588.01 271.78) (xy 591.82 271.78)
 		)
 		(stroke
@@
 	(wire
 		(pts
-			(xy 439.42 96.52) (xy 439.42 99.06)
+			(xy 588.01 276.86) (xy 588.01 279.4)
 		)
 		(stroke
@@
 	(symbol
 		(lib_id "power:GND")
-		(at 439.42 99.06 0)
+		(at 588.01 279.4 0)
 		(unit 1)
 		(exclude_from_sim no)
@@
 		(fields_autoplaced yes)
 		(property "Reference" "#PWR064"
-			(at 439.42 105.41 0)
+			(at 588.01 285.75 0)
 			(effects
 				(font
@@
 		)
 		(property "Value" "GND"
-			(at 439.42 104.14 0)
+			(at 588.01 284.48 0)
 			(effects
 				(font
@@
 		)
 		(property "Footprint" ""
-			(at 439.42 99.06 0)
+			(at 588.01 279.4 0)
 			(effects
 				(font
@@
 		)
 		(property "Datasheet" ""
-			(at 439.42 99.06 0)
+			(at 588.01 279.4 0)
 			(effects
 				(font
@@
 		)
 		(property "Description" "Power symbol creates a global label with name \"GND\" , ground"
-			(at 439.42 99.06 0)
+			(at 588.01 279.4 0)
 			(effects
 				(font
@@
 	(symbol
 		(lib_id "Device:C_Small")
-		(at 439.42 93.98 0)
+		(at 588.01 274.32 0)
 		(unit 1)
 		(exclude_from_sim no)
@@
 		(dnp no)
 		(property "Reference" "C14"
-			(at 436.88 92.964 0)
+			(at 585.47 273.304 0)
 			(effects
 				(font
@@
 		)
 		(property "Value" "10uF"
-			(at 436.88 95.2562 0)
+			(at 585.47 275.5962 0)
 			(effects
 				(font
@@
 		)
 		(property "Footprint" "Capacitor_SMD:C_0402_1005Metric"
-			(at 439.42 93.98 0)
+			(at 588.01 274.32 0)
 			(effects
 				(font
@@
 		)
 		(property "Datasheet" "~"
-			(at 439.42 93.98 0)
+			(at 588.01 274.32 0)
 			(effects
 				(font
@@
 		)
 		(property "Description" "Unpolarized capacitor, small symbol"
-			(at 439.42 93.98 0)
+			(at 588.01 274.32 0)
 			(effects
 				(font
@@
 		)
 		(property "DIGIKEY" "490-GRM155R60J106ME05DCT-ND"
-			(at 439.42 93.98 0)
+			(at 588.01 274.32 0)
 			(effects
 				(font
@@
 	(symbol
 		(lib_id "Device:C_Small")
-		(at 443.23 93.98 0)
+		(at 591.82 274.32 0)
 		(mirror y)
 		(unit 1)
@@
 		(dnp no)
 		(property "Reference" "C15"
-			(at 445.77 92.7162 0)
+			(at 594.36 273.0562 0)
 			(effects
 				(font
@@
 		)
 		(property "Value" "100nF"
-			(at 445.77 95.2562 0)
+			(at 594.36 275.5962 0)
 			(effects
 				(font
@@
 		)
 		(property "Footprint" "Capacitor_SMD:C_0402_1005Metric"
-			(at 443.23 93.98 0)
+			(at 591.82 274.32 0)
 			(effects
 				(font
@@
 		)
 		(property "Datasheet" "~"
-			(at 443.23 93.98 0)
+			(at 591.82 274.32 0)
 			(effects
 				(font
@@
 		)
 		(property "Description" "Unpolarized capacitor, small symbol"
-			(at 443.23 93.98 0)
+			(at 591.82 274.32 0)
 			(effects
 				(font
@@
 		)
 		(property "DIGIKEY" "490-6328-1-ND"
-			(at 443.23 93.98 0)
+			(at 591.82 274.32 0)
 			(effects
 				(font
@@
 	(symbol
 		(lib_id "GameBrian:LFE5U-45F-7BG256x")
-		(at 438.15 115.57 0)
+		(at 586.74 295.91 0)
 		(unit 2)
 		(exclude_from_sim no)
@@
 		(dnp no)
 		(property "Reference" "U1"
-			(at 471.678 178.054 0)
+			(at 620.268 358.394 0)
 			(effects
 				(font
@@
 		)
 		(property "Value" "LFE5U-45F-7BG256x"
-			(at 442.976 178.054 0)
+			(at 591.566 358.394 0)
 			(effects
 				(font
@@
 		)
 		(property "Footprint" "Package_BGA:BGA-256_14.0x14.0mm_Layout16x16_P0.8mm_Ball0.45mm_Pad0.32mm_NSMD"
-			(at 441.96 114.3 0)
+			(at 590.55 294.64 0)
 			(effects
 				(font
@@
 		)
 		(property "Datasheet" "https://www.latticesemi.com/view_document?document_id=50461"
-			(at 441.96 119.38 0)
+			(at 590.55 299.72 0)
 			(effects
 				(font
@@
 		)
 		(property "Description" "ECP5 FPGA, 45K LUTs, 1.2V, BGA-256"
-			(at 438.15 115.57 0)
+			(at 586.74 295.91 0)
 			(effects
 				(font
@@
 		)
 		(property "DIGIKEY" "LFE5U-45F-7BG256C-ND"
-			(at 438.15 115.57 0)
+			(at 586.74 295.91 0)
 			(effects
 				(font
@@
 		(on_board yes)
 		(dnp no)
-		(fields_autoplaced yes)
 		(property "Reference" "U1"
-			(at 379.73 167.6399 0)
+			(at 374.142 219.964 0)
 			(effects
 				(font
@@
 		)
 		(property "Value" "LFE5U-45F-7BG256x"
-			(at 379.73 170.1799 0)
+			(at 335.026 219.964 0)
 			(effects
 				(font
@@
 		(on_board yes)
 		(dnp no)
-		(fields_autoplaced yes)
 		(property "Reference" "U1"
-			(at 360.68 325.1199 0)
+			(at 354.838 359.664 0)
 			(effects
 				(font
@@
 		)
 		(property "Value" "LFE5U-45F-7BG256x"
-			(at 360.68 327.6599 0)
+			(at 310.896 359.664 0)
 			(effects
 				(font
@@
 		(on_board yes)
 		(dnp no)
-		(fields_autoplaced yes)
 		(property "Reference" "U1"
-			(at 543.56 316.2299 0)
+			(at 537.464 368.554 0)
 			(effects
 				(font
@@
 		)
 		(property "Value" "LFE5U-45F-7BG256x"
-			(at 543.56 318.7699 0)
+			(at 496.316 368.554 0)
 			(effects
 				(font
@@
 	(symbol
 		(lib_id "power:+3V3")
-		(at 473.71 91.44 0)
+		(at 622.3 271.78 0)
 		(unit 1)
 		(exclude_from_sim no)
@@
 		(dnp no)
 		(property "Reference" "#PWR052"
-			(at 473.71 95.25 0)
+			(at 622.3 275.59 0)
 			(effects
 				(font
@@
 		)
 		(property "Value" "+3V3"
-			(at 473.71 87.376 0)
+			(at 622.3 267.716 0)
 			(effects
 				(font
@@
 		)
 		(property "Footprint" ""
-			(at 473.71 91.44 0)
+			(at 622.3 271.78 0)
 			(effects
 				(font
@@
 		)
 		(property "Datasheet" ""
-			(at 473.71 91.44 0)
+			(at 622.3 271.78 0)
 			(effects
 				(font
@@
 		)
 		(property "Description" "Power symbol creates a global label with name \"+3V3\""
-			(at 473.71 91.44 0)
+			(at 622.3 271.78 0)
 			(effects
 				(font

Commit message: IDK
Parts:
- J2: footprint GameBrian:GameBoy_GamePak_AGB-002_P1.50mm_Edge_Cuts -> Connector_PinSocket_2.54mm:PinSocket_2x16_P2.54mm_Horizontal
Connections:
- net GBA_A0: now also U1.J15 (PR32B/-/PCLKC2_1/HS/RDQ29)
- net GBA_A1: now also U1.H13 (PR26B/-/HS/RDQ29)
- net GBA_A10: now also U1.F14 (PR14D/-/RDQ17)
- net GBA_A11: now also U1.F15 (PR20C/+/RDQ17)
- net GBA_A12: now also U1.F13 (PR17C/+/RDQ17)
- net GBA_A13: now also U1.F16 (PR23A/+/HS/RDQ29)
- net GBA_A14: now also U1.G12 (PR20A/+/HS/RDQ17)
- net GBA_A15: now also U1.E14 (PR14C/+/RDQ17)
- net GBA_A2: now also U1.H12 (PR26A/+/HS/RDQ29)
- net GBA_A3: now also U1.J16 (PR32A/+/PCLKT2_1/HS/RDQ29)
- net GBA_A4: now also U1.H14 (PR23D/-/RDQ29)
- net GBA_A5: now also U1.H15 (PR29B/-/HS/RDQSN29)
- net GBA_A6: now also U1.G14 (PR23C/+/VREF1_2/RDQ29)
- net GBA_A7: now also U1.G15 (PR23B/-/HS/RDQ29)
- net GBA_A8: now also U1.G13 (PR20B/-/HS/RDQ17)
- net GBA_A9: now also U1.G16 (PR29A/+/GR_PCLK2_1/HS/RDQS29)
- net GBA_CLK: now also U1.K15 (PR32D/-/PCLKC2_0/RDQ29)
- net GBA_D0: now also U1.F12 (PR17D/-/RDQ17)
- net GBA_D1: now also U1.E16 (PR20D/-/RDQ17)
- net GBA_D2: now also U1.E15 (PR17B/-/HS/RDQSN17)
- net GBA_D3: now also U1.D14 (PR11D/-/RDQ17)
- net GBA_D4: now also U1.D16 (PR17A/+/HS/RDQS17)
- net GBA_D5: now also U1.C14 (PR11C/+/RDQ17)
- net GBA_D6: now also U1.C16 (PR14A/+/HS/RDQ17)
- net GBA_D7: now also U1.C15 (PR14B/-/HS/RDQ17)
- net GBA_VDD: now also U1.K14 (PR29D/-/RDQ29)
- net GBA_nCS: now also U1.J14 (PR29C/+/GR_PCLK2_0/RDQ29)
- net GBA_nCS2: now also U1.B16 (PR11A/+/URC_GPLL0T_IN/HS/RDQ17)
- net GBA_nRD: now also U1.K16 (PR32C/+/PCLKT2_0/RDQ29)
- net GBA_nREQ: now also U1.B15 (PR11B/-/URC_GPLL0C_IN/HS/RDQ17)
- net GBA_nWR: now also U1.J13 (PR26C/+/RDQ29)
- net MODE_0: now also U1.N8 (PB15A/+/HOLDN/DI/BUSY/CSSPIN/CEN)
- net MODE_1: now also U1.P8 (PB13B/-/CS1N)
- net USB_DN: now also U1.R6 (PB4B/-/D6/IO6)
- net USB_DP: now also U1.R7 (PB6A/+/D5/MISO2/IO5)
- net USB_PU: now also U1.P7 (PB6B/-/D4/MOSI2/IO4)
Other:
- moved on the sheet: C18, C19, C26, C27, U1D, U1H
